File: cpu-18f4455.sch (EAGLE design)
At the start: 9 parts, among them IC1 PIC18F4455

Commit message: I wired power backwards. I am the dumb. ._.;
Connections:
- removed net ?: IC1.RB0/AN12/INT0/LFT0/SDI/SDA
- removed net N$8: IC1.RB1/AN10/INT1/SCK/SCL
- net +3V3: now also IC1.VDD, IC1.VDD@1; no longer IC1.VSS, IC1.VSS@1
- net GND: now also IC1.VSS, IC1.VSS@1; no longer IC1.VDD, IC1.VDD@1
Changed lines of the file:
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@@
 <instance part="GND1" gate="1" x="17.78" y="121.92"/>
 <instance part="IC1" gate="G$1" x="99.06" y="152.4"/>
-<instance part="+3V2" gate="G$1" x="43.18" y="182.88"/>
-<instance part="+3V3" gate="G$1" x="154.94" y="182.88"/>
+<instance part="+3V2" gate="G$1" x="40.64" y="182.88"/>
+<instance part="+3V3" gate="G$1" x="157.48" y="182.88"/>
 <instance part="GND2" gate="1" x="43.18" y="116.84"/>
 <instance part="GND3" gate="1" x="154.94" y="111.76"/>
@@
 <segment>
 <pinref part="GND2" gate="1" pin="GND"/>
-<pinref part="IC1" gate="G$1" pin="VDD"/>
-<wire x1="43.18" y1="119.38" x2="43.18" y2="162.56" width="0.1524" layer="91"/>
-<wire x1="43.18" y1="162.56" x2="63.5" y2="162.56" width="0.1524" layer="91"/>
-<label x="48.26" y="162.56" size="1.778" layer="95"/>
-</segment>
-<segment>
-<pinref part="IC1" gate="G$1" pin="VDD@1"/>
-<wire x1="134.62" y1="137.16" x2="154.94" y2="137.16" width="0.1524" layer="91"/>
+<wire x1="43.18" y1="119.38" x2="43.18" y2="165.1" width="0.1524" layer="91"/>
+<pinref part="IC1" gate="G$1" pin="VSS"/>
+<wire x1="43.18" y1="165.1" x2="63.5" y2="165.1" width="0.1524" layer="91"/>
+</segment>
+<segment>
 <pinref part="GND3" gate="1" pin="GND"/>
-<wire x1="154.94" y1="137.16" x2="154.94" y2="114.3" width="0.1524" layer="91"/>
-<label x="137.16" y="137.16" size="1.778" layer="95"/>
+<wire x1="154.94" y1="139.7" x2="154.94" y2="114.3" width="0.1524" layer="91"/>
+<pinref part="IC1" gate="G$1" pin="VSS@1"/>
+<wire x1="134.62" y1="139.7" x2="154.94" y2="139.7" width="0.1524" layer="91"/>
 </segment>
 <segment>
@@
 </segment>
 <segment>
-<pinref part="IC1" gate="G$1" pin="VSS"/>
-<wire x1="63.5" y1="165.1" x2="43.18" y2="165.1" width="0.1524" layer="91"/>
 <pinref part="+3V2" gate="G$1" pin="+3V3"/>
-<wire x1="43.18" y1="165.1" x2="43.18" y2="180.34" width="0.1524" layer="91"/>
-<label x="48.26" y="165.1" size="1.778" layer="95"/>
-</segment>
-<segment>
-<pinref part="IC1" gate="G$1" pin="VSS@1"/>
-<wire x1="134.62" y1="139.7" x2="154.94" y2="139.7" width="0.1524" layer="91"/>
+<wire x1="40.64" y1="162.56" x2="40.64" y2="180.34" width="0.1524" layer="91"/>
+<pinref part="IC1" gate="G$1" pin="VDD"/>
+<wire x1="63.5" y1="162.56" x2="40.64" y2="162.56" width="0.1524" layer="91"/>
+</segment>
+<segment>
 <pinref part="+3V3" gate="G$1" pin="+3V3"/>
-<wire x1="154.94" y1="139.7" x2="154.94" y2="180.34" width="0.1524" layer="91"/>
-<label x="137.16" y="139.7" size="1.778" layer="95"/>
+<wire x1="157.48" y1="137.16" x2="157.48" y2="180.34" width="0.1524" layer="91"/>
+<pinref part="IC1" gate="G$1" pin="VDD@1"/>
+<wire x1="134.62" y1="137.16" x2="157.48" y2="137.16" width="0.1524" layer="91"/>
 </segment>
 <segment>
@@
 </segment>
 </net>
-<net name="N$8" class="0">
-<segment>
-<pinref part="IC1" gate="G$1" pin="RB1/AN10/INT1/SCK/SCL"/>
-<wire x1="45.72" y1="157.48" x2="63.5" y2="157.48" width="0.1524" layer="91"/>
-<label x="48.26" y="157.48" size="1.778" layer="95"/>
-</segment>
-</net>
-<net name="?" class="0">
-<segment>
-<pinref part="IC1" gate="G$1" pin="RB0/AN12/INT0/LFT0/SDI/SDA"/>
-<wire x1="63.5" y1="160.02" x2="45.72" y2="160.02" width="0.1524" layer="91"/>
-<label x="48.26" y="160.02" size="1.778" layer="95"/>
-</segment>
-</net>
